Commit message: fix: urdf mesh paths

File: projects/piper_urdf/urdf/piper.urdf (robot description, URDF)
Before this commit: robot piper_fl, 9 links, 8 joints
Links:
- link fl_base_link: geometry collision mesh filename=../meshes/base_link.STL; visual mesh filename=../meshes/base_link.dae
- link fl_link1: geometry collision mesh filename=../meshes/link1.STL; visual mesh filename=../meshes/link1.dae
- link fl_link2: geometry collision mesh filename=../meshes/link2.STL; visual mesh filename=../meshes/link2.dae
- link fl_link3: geometry collision mesh filename=../meshes/link3.STL; visual mesh filename=../meshes/link3.dae
- link fl_link4: geometry collision mesh filename=../meshes/link4.STL; visual mesh filename=../meshes/link4.dae
- link fl_link5: geometry collision mesh filename=../meshes/link5.STL; visual mesh filename=../meshes/link5.dae
- link fl_link6: geometry collision mesh filename=../meshes/link6.STL; visual mesh filename=../meshes/link6.dae
- link fl_link7: geometry collision mesh filename=../meshes/link7.STL; visual mesh filename=../meshes/link7.dae
- link fl_link8: geometry collision mesh filename=../meshes/link8.STL; visual mesh filename=../meshes/link8.dae
